File: Elec/drive.kicad_sch (KiCad schematic)
At the start: 70 parts, among them J1 PSU, J2 Conn_01x40, J3 Comm_Conn1, J4 Comm_Conn2, U2 DRV8313PWPR, U3 DRV8313PWPR, U4 DRV8313PWPR, U5 DRV8313PWPR, U6 DRV8313PWPR, U7 DRV8313PWPR, U8 DRV8313PWPR

Commit message: Correcting UC symbol
+ added connections
Parts:
- added C47: C, symbol Device:C
- added R8: 10k, symbol Device:R
- added SW1: SW_SPST, symbol Switch:SW_SPST
Connections:
- net +3.3V: now also C47.1, R8.1
- net +3.3VA: now also U1.19 (AVDD); no longer U1.25 (AVDD)
- net +3V3: now also U1.10 (VDD), U1.25 (VDD), U1.40 (VSS), U1.57 (VDD); no longer U1.12 (VDD), U1.31 (VDD), U1.51 (VDD), U1.71 (VDD)
- net DATA_M1-2: now also U1.21 (RD12)
- net DATA_M3-4: now also U1.23 (RC2)
- net DATA_M5-6: now also U1.27 (RC3)
- net DATA_M7: now also U1.29 (RB1)
- net GND: now also U1.20 (AVSS), U1.40 (VSS), U1.56 (VSS), U1.9 (VSS), SW1.1 (A); no longer U1.11 (VSS), U1.32 (VSS), U1.50 (VSS), U1.70 (VSS)
- net M1_EN1: now also U1.55 (RD3)
- net M1_EN2: now also U1.54 (RD4)
- net M1_EN3: now also U1.53 (RC11)
- net M2_EN1: now also U1.52 (RC10)
- net M2_EN2: now also U1.51 (RC5)
- net M2_EN3: now also U1.50 (RC4)
- net M3_EN1: now also U1.49 (RB9)
- net M3_EN2: now also U1.48 (RB8)
- net M3_EN3: now also U1.47 (RB7)
- net M4_EN1: now also U1.46 (RB6)
- net M4_EN2: now also U1.45 (RB5)
- net M4_EN3: now also U1.44 (RD5)
- net M5_EN1: now also U1.43 (RD6)
- net M5_EN2: now also U1.42 (RD7)
- net M5_EN3: now also U1.39 (RD8)
- net M6_EN1: now also U1.38 (RD9)
- net M6_EN2: now also U1.37 (RC9)
- net M6_EN3: now also U1.36 (RC8)
- net M7_EN1: now also U1.35 (RB4)
- net M7_EN2: now also U1.34 (RB3)
- net M7_EN3: now also U1.33 (RB2)
- net Rx1: now also U1.15 (RA1)
- net Rx2: now also U1.17 (RA3)
- net SEQ_Update_M1-2: now also U1.18 (RA4)
- net SEQ_Update_M3-4: now also U1.22 (RC1)
- net SEQ_Update_M5-6: now also U1.24 (RC6)
- net SEQ_Update_M7: now also U1.28 (RB0)
- net Serial_CLK: now also U1.58 (RD2)
- net Tx1: now also U1.14 (RA0)
- net Tx2: now also U1.16 (RA2)
- net /Fault_1: now also U1.1 (RB14); no longer R2.2, R3.2, R4.2, R5.2, R6.2, R7.2, U3.18 (FAULT_N), U4.18 (FAULT_N), U5.18 (FAULT_N), U6.18 (FAULT_N), U7.18 (FAULT_N), U8.18 (FAULT_N)
- net /Reset: now also U1.60 (RD0)
- net /Sleep: now also U1.59 (RD1)
- net /Fault_3: now reaches U1.3 (RC12)
- net /Fault_3: now also R3.2, U4.18 (FAULT_N)
- net /Fault_4: now reaches U1.4 (RC13)
- net /Fault_4: now also R4.2, U5.18 (FAULT_N)
- net /Fault_5: now reaches U1.5 (RC14)
- net /Fault_5: now also R5.2, U6.18 (FAULT_N)
- net /Fault_6: now reaches U1.6 (RC15)
- net /Fault_6: now also R6.2, U7.18 (FAULT_N)
- net Mem_clr: now reaches U1.7 (MCLR)
- net Mem_clr: now also C47.2, R8.2, SW1.2 (B)
- net /Fault_7: now reaches U1.8 (RD15)
- net /Fault_7: now also R7.2, U8.18 (FAULT_N)
- net /E renamed /Fault_2
- net /Fault_2: now also R2.2, U3.18 (FAULT_N)

Commit message: Added a FPGA and a TODO list
The FPGA will be used to interpret strobe encoder signals
Parts:
- added C48: 0.01u, symbol Device:C
- added C49: 0.1u, symbol Device:C
- added C50: 0.47u, symbol Device:C
- added C51, C53: 10uF, symbol Device:C
- added C52: 0.1uF, symbol Device:C
- added J10: M6, symbol Connector_Generic:Conn_01x03
- added J11: M7, symbol Connector_Generic:Conn_01x03
- added J5: M1, symbol Connector_Generic:Conn_01x03
- added J6: M2, symbol Connector_Generic:Conn_01x03
- added J7: M3, symbol Connector_Generic:Conn_01x03
- added J8: M4, symbol Connector_Generic:Conn_01x03
- added J9: M5, symbol Connector_Generic:Conn_01x03
- added R10, R11, R12: 10k, symbol Device:R
- added R13: 20k, symbol Device:R
- added R9: 1k, symbol Device:R
- added SW3: FPGA reset, symbol Switch:SW_SPDT
- added U13: ICE40LP384-SG32, QFNS32_LAT, symbol ICE40LP384-SG32:ICE40LP384-SG32
- added U14: DRV8313PWPR, PWP0028F_N, symbol DRV8313PWPR:DRV8313PWPR
- C47: value C -> 10uF
- J2: value Conn_01x40 -> Debug Conn
- SW1: value SW_SPST -> Uc mem CLR
Connections:
- net +3.3V: now also C53.1, SW3.1 (A), U13.16 (VCC_SPI), U13.17 (VCCIO_1), U13.25 (VCC), U13.28 (VCCIO_0), U13.4 (VCCIO_3), U13.9 (VCCIO_2)
- net +3V3: now also C52.1, R10.1, R12.1
- net GND: now also C50.1, R11.2, R13.1, U13.21 (GND), U13.3 (GND), U14.12 (COMPP), U14.13 (COMPN), U14.14 (GND), U14.19 (COMPO_N), U14.20 (GND), U14.21 (NC), U14.28 (GND), U14.29 (PAD)
- net GND1: now also C51.2, C52.2, U14.10 (PGND3), U14.6 (PGND1), U14.7 (PGND2)
- net M1_1: now also J5.1 (Pin_1)
- net M1_2: now also J5.2 (Pin_2)
- net M1_3: now also J5.3 (Pin_3)
- net M1_EN1: now also U1.60 (RD0); no longer U1.55 (RD3)
- net M1_EN2: now also U1.59 (RD1); no longer U1.54 (RD4)
- net M1_EN3: now also U1.58 (RD2); no longer U1.53 (RC11)
- net M2_1: now also J6.1 (Pin_1)
- net M2_2: now also J6.2 (Pin_2)
- net M2_3: now also J6.3 (Pin_3)
- net M2_EN1: now also U1.55 (RD3); no longer U1.52 (RC10)
- net M2_EN2: now also U1.54 (RD4); no longer U1.51 (RC5)
- net M2_EN3: now also U1.53 (RC11); no longer U1.50 (RC4)
- net M3_1: now also J7.1 (Pin_1)
- net M3_2: now also J7.2 (Pin_2)
- net M3_3: now also J7.3 (Pin_3)
- net M3_EN1: now also U1.52 (RC10); no longer U1.49 (RB9)
- net M3_EN2: now also U1.51 (RC5); no longer U1.48 (RB8)
- net M3_EN3: now also U1.50 (RC4); no longer U1.47 (RB7)
- net M4_1: now also J8.1 (Pin_1)
- net M4_2: now also J8.2 (Pin_2)
- net M4_3: now also J8.3 (Pin_3)
- net M4_EN1: now also U1.49 (RB9); no longer U1.46 (RB6)
- net M4_EN2: now also U1.48 (RB8); no longer U1.45 (RB5)
- net M4_EN3: now also U1.47 (RB7); no longer U1.44 (RD5)
- net M5_1: now also J9.1 (Pin_1)
- net M5_2: now also J9.2 (Pin_2)
- net M5_3: now also J9.3 (Pin_3)
- net M5_EN1: now also U1.46 (RB6); no longer U1.43 (RD6)
- net M5_EN2: now also U1.45 (RB5); no longer U1.42 (RD7)
- net M5_EN3: now also U1.44 (RD5); no longer U1.39 (RD8)
- net M6_1: now also J10.1 (Pin_1)
- net M6_2: now also J10.2 (Pin_2)
- net M6_3: now also J10.3 (Pin_3)
- net M6_EN1: now also U1.43 (RD6); no longer U1.38 (RD9)
- net M6_EN2: now also U1.42 (RD7); no longer U1.37 (RC9)
- net M6_EN3: now also U1.39 (RD8); no longer U1.36 (RC8)
- net M7_1: now also J11.1 (Pin_1)
- net M7_2: now also J11.2 (Pin_2)
- net M7_3: now also J11.3 (Pin_3)
- net M7_EN1: now also U1.38 (RD9); no longer U1.35 (RB4)
- net M7_EN2: now also U1.37 (RC9); no longer U1.34 (RB3)
- net M7_EN3: now also U1.36 (RC8); no longer U1.33 (RB2)
- net Serial_CLK: now also U1.61 (RB10); no longer U1.58 (RD2)
- net Vdrive: now also C49.2, C51.1, U14.11 (VM), U14.4 (VM)
- net /Reset: now also U1.63 (RB12), R12.2, U14.16 (RESET_N); no longer U1.60 (RD0)
- net /Sleep: now also U1.62 (RB11), R11.1, U14.17 (SLEEP_N); no longer U1.59 (RD1)
- net /Fault_8: now reaches U1.11 (RD14)
- net /Fault_8: now also R10.2, U14.18 (FAULT_N)
- net FPGA_Reset: now reaches U1.64 (RB13)
- net FPGA_Reset: now also R9.1
- net M8_P3: now reaches U12.13 (Q5)
- net M8_P3: now also U14.23 (IN3)
- net M8_P2: now reaches U12.14 (Q4)
- net M8_P2: now also U14.25 (IN2)
- net M8_P1: now reaches U12.7 (Q3)
- net M8_P1: now also U14.27 (IN1)
- net DATA_M7 renamed DATA_M7-8
- net SEQ_Update_M7 renamed SEQ_Update_M7-8
- new net: C53.2, R13.2, SW3.2 (B), U13.10 (CRESET_B)
- new net: R9.2, SW3.3 (C)
- new net: C50.2, U14.15 (V3P3OUT)
- new net: C48.1, U14.1 (CP1)
- new net: C48.2, U14.2 (CP2)
- new net: C49.1, U14.3 (VCP)
- new net M8_1: U14.5 (OUT1)
- new net M8_2: U14.8 (OUT2)
- new net M8_3: U14.9 (OUT3)
- new net M8_EN1: U1.35 (RB4), U14.26 (EN1)
- new net M8_EN2: U1.34 (RB3), U14.24 (EN2)
- new net M8_EN3: U1.33 (RB2), U14.22 (EN3)
- no-connect marks 19 -> 18
Other:
- note added: "8 motors Candidates: - 42SHDC3025-24B : Step motor, requires 1 drive per motor. Set Vref to 1.056v - DRV8313PWPR : BLDC , requires 1 drive and 3 PWM per motor"
- note added: "TODO: - Finding a fitting connector for the motor phases (terminal block?) - Connecting the FPGA to the MCU (SPI and control signals) - Connecting a programming interface for the MCU and FPGA for external programming - Connecting the bebug header (choose witch signals are important) - Adding test points - FPGA Power supply and decoupling - Add a connector for each SR outpouts (1 per SR)"
- note removed: "7 motors Candidates: - 42SHDC3025-24B : Step motor, requires 1 drive per motor. Set Vref to 1.056v - DRV8313PWPR : BLDC , requires 1 drive and 3 PWM per motor"
- moved on the sheet: C10, C11, C12, C13, C14, C15, C16, C17, C18, C19, C20, C21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
